File: Ref_V.sch (KiCad schematic (older format))
At the start: 8 parts, among them U1 LM4041DYM3-ADJ-TR, U2 LM4041DYM3-ADJ-TR

Commit message: Fixed some mistakes of v0.1
Connections:
- wire segments 32 -> 28
Changed lines of the file:
@@
 Comment4 ""
 $EndDescr
-Text HLabel 5800 4550 2    50   Output ~ 0
+Text HLabel 5800 5150 2    50   Output ~ 0
 Ref_V-
-Text HLabel 5800 3350 2    50   Output ~ 0
+Text HLabel 5800 3650 2    50   Output ~ 0
 Ref_V+
 Text HLabel 3700 2600 0    50   Input ~ 0
@@
 L Reference_Voltage:LM4041LP-ADJ U1
 U 1 1 5DD703A3
-P 4750 3650
-F 0 "U1" V 4796 3563 50  0000 R CNN
-F 1 "LM4041DYM3-ADJ-TR" V 4705 3563 50  0000 R CNN
-F 2 "Package_TO_SOT_SMD:SOT-23" H 4750 3450 50  0001 C CIN
-F 3 "http://www.ti.com/lit/ds/symlink/lm4041-n.pdf" H 4850 3800 50  0001 C CIN
-	1    4750 3650
+P 4750 3350
+F 0 "U1" V 4796 3263 50  0000 R CNN
+F 1 "LM4041DYM3-ADJ-TR" V 4705 3263 50  0000 R CNN
+F 2 "Package_TO_SOT_SMD:SOT-23" H 4750 3150 50  0001 C CIN
+F 3 "http://www.ti.com/lit/ds/symlink/lm4041-n.pdf" H 4850 3500 50  0001 C CIN
+	1    4750 3350
 	0    1    -1   0
 $EndComp
-Wire Wire Line
-	4750 3800 4750 3950
 $Comp
 L Device:R_Small R?
 U 1 1 5DD730FE
-P 4750 3200
+P 4750 3800
 AR Path="/5DCD3ADE/5DD730FE" Ref="R?"  Part="1"
 AR Path="/5DCD39AB/5DD730FE" Ref="R?"  Part="1"
 AR Path="/5DD2EEC0/5DD730FE" Ref="R27"  Part="1"
-F 0 "R27" V 4554 3200 50  0000 C CNN
-F 1 "470R" V 4645 3200 50  0000 C CNN
-F 2 "Resistor_SMD:R_0805_2012Metric" H 4750 3200 50  0001 C CNN
-F 3 "~" H 4750 3200 50  0001 C CNN
-	1    4750 3200
+F 0 "R27" V 4554 3800 50  0000 C CNN
+F 1 "470R" V 4645 3800 50  0000 C CNN
+F 2 "Resistor_SMD:R_0805_2012Metric" H 4750 3800 50  0001 C CNN
+F 3 "~" H 4750 3800 50  0001 C CNN
+	1    4750 3800
 	1    0    0    -1
 $EndComp
-Wire Wire Line
-	4750 3100 4750 3050
 $Comp
 L Device:R_Small R?
 U 1 1 5DD7390A
-P 5150 3500
+P 5150 3200
 AR Path="/5DCD3ADE/5DD7390A" Ref="R?"  Part="1"
 AR Path="/5DCD39AB/5DD7390A" Ref="R?"  Part="1"
 AR Path="/5DD2EEC0/5DD7390A" Ref="R29"  Part="1"
-F 0 "R29" V 4954 3500 50  0000 C CNN
-F 1 "3k" V 5045 3500 50  0000 C CNN
+F 0 "R29" V 4954 3200 50  0000 C CNN
+F 1 "3k" V 5045 3200 50  0000 C CNN
+F 2 "Resistor_SMD:R_0805_2012Metric" H 5150 3200 50  0001 C CNN
+F 3 "~" H 5150 3200 50  0001 C CNN
+	1    5150 3200
+	-1   0    0    1
+$EndComp
+$Comp
+L Device:R_Small R?
+U 1 1 5DD73DBA
+P 5150 3500
+AR Path="/5DCD3ADE/5DD73DBA" Ref="R?"  Part="1"
+AR Path="/5DCD39AB/5DD73DBA" Ref="R?"  Part="1"
+AR Path="/5DD2EEC0/5DD73DBA" Ref="R30"  Part="1"
+F 0 "R30" V 4954 3500 50  0000 C CNN
+F 1 "8.2k" V 5045 3500 50  0000 C CNN
 F 2 "Resistor_SMD:R_0805_2012Metric" H 5150 3500 50  0001 C CNN
 F 3 "~" H 5150 3500 50  0001 C CNN
@@
 	-1   0    0    1
 $EndComp
-$Comp
-L Device:R_Small R?
-U 1 1 5DD73DBA
-P 5150 3800
-AR Path="/5DCD3ADE/5DD73DBA" Ref="R?"  Part="1"
-AR Path="/5DCD39AB/5DD73DBA" Ref="R?"  Part="1"
-AR Path="/5DD2EEC0/5DD73DBA" Ref="R30"  Part="1"
-F 0 "R30" V 4954 3800 50  0000 C CNN
-F 1 "8.2k" V 5045 3800 50  0000 C CNN
-F 2 "Resistor_SMD:R_0805_2012Metric" H 5150 3800 50  0001 C CNN
-F 3 "~" H 5150 3800 50  0001 C CNN
-	1    5150 3800
-	-1   0    0    1
-$EndComp
-Wire Wire Line
-	4750 3300 4750 3350
-Wire Wire Line
-	5150 3350 4750 3350
-Connection ~ 4750 3350
-Wire Wire Line
-	4750 3350 4750 3500
-Wire Wire Line
-	5150 3700 5150 3650
-Wire Wire Line
-	4950 3650 5150 3650
-Connection ~ 5150 3650
-Wire Wire Line
-	5150 3650 5150 3600
-Wire Wire Line
-	5150 3950 4950 3950
-Wire Wire Line
-	5150 3900 5150 3950
-Wire Wire Line
-	5150 3350 5150 3400
-Wire Wire Line
-	5150 3350 5800 3350
+Wire Wire Line
+	4750 3000 4750 3050
+Wire Wire Line
+	5150 3050 4750 3050
+Connection ~ 4750 3050
+Wire Wire Line
+	4750 3050 4750 3200
+Wire Wire Line
+	5150 3400 5150 3350
+Wire Wire Line
+	4950 3350 5150 3350
 Connection ~ 5150 3350
+Wire Wire Line
+	5150 3350 5150 3300
+Wire Wire Line
+	5150 3050 5150 3100
+Wire Wire Line
+	5150 3650 5800 3650
 $Comp
 L Reference_Voltage:LM4041LP-ADJ U2
@@
 	0    1    -1   0
 $EndComp
-Wire Wire Line
-	4750 5000 4750 5150
-$Comp
-L Device:R_Small R?
-U 1 1 5DD784E5
-P 4750 4400
-AR Path="/5DCD3ADE/5DD784E5" Ref="R?"  Part="1"
-AR Path="/5DCD39AB/5DD784E5" Ref="R?"  Part="1"
-AR Path="/5DD2EEC0/5DD784E5" Ref="R28"  Part="1"
-F 0 "R28" V 4554 4400 50  0000 C CNN
-F 1 "470R" V 4645 4400 50  0000 C CNN
-F 2 "Resistor_SMD:R_0805_2012Metric" H 4750 4400 50  0001 C CNN
-F 3 "~" H 4750 4400 50  0001 C CNN
-	1    4750 4400
-	1    0    0    -1
-$EndComp
-Wire Wire Line
-	4750 4300 4750 4250
 $Comp
 L Device:R_Small R?
@@
 	5150 4850 5150 4800
 Wire Wire Line
-	5150 5150 4950 5150
-Wire Wire Line
-	5150 5100 5150 5150
-Wire Wire Line
 	5150 4550 5150 4600
 Wire Wire Line
-	5150 4550 5800 4550
-Connection ~ 5150 4550
-Text Notes 5850 3250 0    50   ~ 0
+	5150 5150 5800 5150
+Text Notes 5850 3550 0    50   ~ 0
 -0.4V
-Text Notes 5750 4750 0    50   ~ 0
+Text Notes 5750 5350 0    50   ~ 0
 -2.6V
-Text Notes 6000 4050 0    50   ~ 0
+Text Notes 5800 4300 0    50   ~ 0
 Vo = 1.233 * (R2/R1 + 1)\n\nR2/R1 = (V0 / 1.233) - 1
 $Comp
@@
 L power:GND #PWR?
 U 1 1 5DD7D9C6
-P 4900 3050
+P 4750 3000
 AR Path="/5DD7D9C6" Ref="#PWR?"  Part="1"
 AR Path="/5DD2EEC0/5DD7D9C6" Ref="#PWR0162"  Part="1"
-F 0 "#PWR0162" H 4900 2800 50  0001 C CNN
-F 1 "GND" H 4905 2877 50  0001 C CNN
-F 2 "" H 4900 3050 50  0001 C CNN
-F 3 "" H 4900 3050 50  0001 C CNN
-	1    4900 3050
-	1    0    0    -1
+F 0 "#PWR0162" H 4750 2750 50  0001 C CNN
+F 1 "GND" H 4755 2827 50  0001 C CNN
+F 2 "" H 4750 3000 50  0001 C CNN
+F 3 "" H 4750 3000 50  0001 C CNN
+	1    4750 3000
+	-1   0    0    1
 $EndComp
 Wire Wire Line
 	3850 2900 3700 2900
-Wire Wire Line
-	4900 3050 4750 3050
-$Comp
-L power:GND #PWR?
-U 1 1 5DD80ADE
-P 4900 4250
-AR Path="/5DD80ADE" Ref="#PWR?"  Part="1"
-AR Path="/5DD2EEC0/5DD80ADE" Ref="#PWR0163"  Part="1"
-F 0 "#PWR0163" H 4900 4000 50  0001 C CNN
-F 1 "GND" H 4905 4077 50  0001 C CNN
-F 2 "" H 4900 4250 50  0001 C CNN
-F 3 "" H 4900 4250 50  0001 C CNN
-	1    4900 4250
-	1    0    0    -1
-$EndComp
-Wire Wire Line
-	4900 4250 4750 4250
 $Comp
 L power:-5V #PWR?
 U 1 1 5DD81409
-P 4950 4000
+P 4750 3950
 AR Path="/5DD81409" Ref="#PWR?"  Part="1"
 AR Path="/5DD2EEC0/5DD81409" Ref="#PWR0164"  Part="1"
-F 0 "#PWR0164" H 4950 4100 50  0001 C CNN
-F 1 "-5V" H 4800 4050 50  0000 C CNN
-F 2 "" H 4950 4000 50  0001 C CNN
-F 3 "" H 4950 4000 50  0001 C CNN
-	1    4950 4000
-	-1   0    0    1
-$EndComp
-Wire Wire Line
-	4950 4000 4950 3950
-Connection ~ 4950 3950
-Wire Wire Line
-	4950 3950 4750 3950
-$Comp
-L power:-5V #PWR?
-U 1 1 5DD81BA9
-P 4950 5200
-AR Path="/5DD81BA9" Ref="#PWR?"  Part="1"
-AR Path="/5DD2EEC0/5DD81BA9" Ref="#PWR0165"  Part="1"
-F 0 "#PWR0165" H 4950 5300 50  0001 C CNN
-F 1 "-5V" H 4800 5250 50  0000 C CNN
-F 2 "" H 4950 5200 50  0001 C CNN
-F 3 "" H 4950 5200 50  0001 C CNN
-	1    4950 5200
-	-1   0    0    1
-$EndComp
-Wire Wire Line
-	4950 5150 4950 5200
-Connection ~ 4950 5150
-Wire Wire Line
-	4950 5150 4750 5150
+F 0 "#PWR0164" H 4750 4050 50  0001 C CNN
+F 1 "-5V" H 4600 4000 50  0000 C CNN
+F 2 "" H 4750 3950 50  0001 C CNN
+F 3 "" H 4750 3950 50  0001 C CNN
+	1    4750 3950
+	-1   0    0    1
+$EndComp
 $Comp
 L power:GND #PWR?
@@
 	1    0    0    -1
 $EndComp
-Text Notes 5450 3500 0    50   ~ 0
+Text Notes 5450 3200 0    50   ~ 0
 R1
-Text Notes 5450 3850 0    50   ~ 0
+Text Notes 5450 3550 0    50   ~ 0
 R2
 Text Notes 5450 4700 0    50   ~ 0
@@
 Text Notes 5450 5050 0    50   ~ 0
 R2
+$Comp
+L power:GND #PWR?
+U 1 1 5DD80ADE
+P 4750 4500
+AR Path="/5DD80ADE" Ref="#PWR?"  Part="1"
+AR Path="/5DD2EEC0/5DD80ADE" Ref="#PWR0163"  Part="1"
+F 0 "#PWR0163" H 4750 4250 50  0001 C CNN
+F 1 "GND" H 4755 4327 50  0001 C CNN
+F 2 "" H 4750 4500 50  0001 C CNN
+F 3 "" H 4750 4500 50  0001 C CNN
+	1    4750 4500
+	-1   0    0    1
+$EndComp
+$Comp
+L Device:R_Small R?
+U 1 1 5DD784E5
+P 4750 5300
+AR Path="/5DCD3ADE/5DD784E5" Ref="R?"  Part="1"
+AR Path="/5DCD39AB/5DD784E5" Ref="R?"  Part="1"
+AR Path="/5DD2EEC0/5DD784E5" Ref="R28"  Part="1"
+F 0 "R28" V 4554 5300 50  0000 C CNN
+F 1 "470R" V 4645 5300 50  0000 C CNN
+F 2 "Resistor_SMD:R_0805_2012Metric" H 4750 5300 50  0001 C CNN
+F 3 "~" H 4750 5300 50  0001 C CNN
+	1    4750 5300
+	1    0    0    -1
+$EndComp
+$Comp
+L power:-5V #PWR?
+U 1 1 5DD81BA9
+P 4750 5450
+AR Path="/5DD81BA9" Ref="#PWR?"  Part="1"
+AR Path="/5DD2EEC0/5DD81BA9" Ref="#PWR0165"  Part="1"
+F 0 "#PWR0165" H 4750 5550 50  0001 C CNN
+F 1 "-5V" H 4600 5500 50  0000 C CNN
+F 2 "" H 4750 5450 50  0001 C CNN
+F 3 "" H 4750 5450 50  0001 C CNN
+	1    4750 5450
+	-1   0    0    1
+$EndComp
+Wire Wire Line
+	5150 5100 5150 5150
+Connection ~ 5150 3650
+Wire Wire Line
+	4750 3500 4750 3650
+Wire Wire Line
+	5150 3600 5150 3650
+Wire Wire Line
+	4750 3900 4750 3950
+Wire Wire Line
+	4750 3700 4750 3650
+Connection ~ 5150 5150
+Wire Wire Line
+	4750 5150 4750 5200
+Wire Wire Line
+	4750 5150 4750 5000
+Wire Wire Line
+	4750 5400 4750 5450
+Connection ~ 4750 5150
+Wire Wire Line
+	4750 5150 5150 5150
+Connection ~ 4750 3650
+Wire Wire Line
+	4750 3650 5150 3650
 $EndSCHEMATC
