File: Ref_V.sch (KiCad schematic (older format))
At the start: 8 parts, among them U1 LM4041DYM3-ADJ-TR, U2 LM4041DYM3-ADJ-TR

Commit message: Changed: voltage ref to use one regulator
Parts:
- removed R30: 8.2k, Resistor_SMD:R_0805_2012Metric, symbol Device:R_Small
- removed U1: LM4041DYM3-ADJ-TR, Package_TO_SOT_SMD:SOT-23, symbol Reference_Voltage:LM4041LP-ADJ
- R27: value 470R -> 1k
- R29: value 3k -> 200R
- R31: value 8.2k -> 6.8k
Connections:
- wire segments 28 -> 21
